File: PCB/smartwatch.kicad_pcb (KiCad board)
At the start: 2 copper layers, 37 x 23.5 mm, 66 parts, among them U1 STM32F103C8T6, U2 HM-10_MIN, U3 M25P40, U4 BMC150, U5 BMP180, U6 STC4054, U7 NCP551, U8 SH1106, X1 VIN, X10 3V3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

Commit message: Values update
Parts:
- C1, C2, C3, C4: value capacitor -> 15p
- C6, C7: value capacitor -> 0.1
- R1: value resistor -> 10k
- R12, R13: value resistor -> 1k
- R14, R15: value 390k -> 10k
- R2, R4, R6, R7: value resistor -> 100
- R3: value resistor -> 100k
- XC2: value CRYSTAL_2pin -> 32768
Changed lines of the file:
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@@
-(kicad_pcb (version 4) (host pcbnew "(2016-04-05 BZR 6665, Git e1b308b)-product")
+(kicad_pcb (version 4) (host pcbnew "(2016-04-26 BZR 6712, Git b92ad6f)-product")
   (general
     (links 193)
     (no_connects 0)
-    (area 169.233572 77.815476 214.1925 108.866428)
+    (area 173.924999 80.424999 211.075001 104.075001)
     (thickness 0.6)
     (drawings 16)
@@
   (module SO:SO8 (layer F.Cu)
     (at 200.5 82.6 270)
-    (fp_text reference U3 (at 0.7 -3 360) (layer F.SilkS) hide
+    (fp_text reference U3 (at 0.7 -3) (layer F.SilkS) hide
       (effects (font (size 0.8 0.8) (thickness 0.16)))
     )
@@
   (module CRYSTAL:SMD_3215 (layer F.Cu)
     (at 196.2 100.1 270)
-    (fp_text reference XC2 (at -1.25 0.5 360) (layer F.SilkS) hide
+    (fp_text reference XC2 (at -1.25 0.5) (layer F.SilkS) hide
       (effects (font (size 1 1) (thickness 0.2)))
     )
-    (fp_text value CRYSTAL_2pin (at 0.9 -3.3 270) (layer F.Fab) hide
+    (fp_text value 32768 (at 0.9 -3.3 270) (layer F.Fab) hide
       (effects (font (size 1 1) (thickness 0.15)))
     )
@@
       (effects (font (size 0.5 0.5) (thickness 0.125)))
     )
-    (fp_text value resistor (at 0.6 1.7 90) (layer F.Fab) hide
+    (fp_text value 10k (at 0.6 1.7 90) (layer F.Fab) hide
       (effects (font (size 1 1) (thickness 0.15)))
     )
@@
       (effects (font (size 0.5 0.5) (thickness 0.125)))
     )
-    (fp_text value capacitor (at 0.6 1.7 90) (layer F.Fab) hide
+    (fp_text value 15p (at 0.6 1.7 90) (layer F.Fab) hide
       (effects (font (size 1 1) (thickness 0.15)))
     )
@@
       (effects (font (size 0.5 0.5) (thickness 0.125)))
     )
-    (fp_text value capacitor (at 0.6 1.7 270) (layer F.Fab) hide
+    (fp_text value 15p (at 0.6 1.7 270) (layer F.Fab) hide
       (effects (font (size 1 1) (thickness 0.15)))
     )
@@
       (effects (font (size 0.5 0.5) (thickness 0.125)))
     )
-    (fp_text value capacitor (at 0.6 1.7) (layer F.Fab) hide
+    (fp_text value 15p (at 0.6 1.7) (layer F.Fab) hide
       (effects (font (size 1 1) (thickness 0.15)))
     )
@@
       (effects (font (size 0.5 0.5) (thickness 0.125)))
     )
-    (fp_text value capacitor (at 0.6 1.7 90) (layer F.Fab) hide
+    (fp_text value 15p (at 0.6 1.7 90) (layer F.Fab) hide
       (effects (font (size 1 1) (thickness 0.15)))
     )
@@
       (effects (font (size 0.5 0.5) (thickness 0.125)))
     )
-    (fp_text value resistor (at 0.6 1.7 90) (layer F.Fab) hide
+    (fp_text value 100 (at 0.6 1.7 90) (layer F.Fab) hide
       (effects (font (size 1 1) (thickness 0.15)))
     )
@@
       (effects (font (size 0.5 0.5) (thickness 0.125)))
     )
-    (fp_text value resistor (at 0.6 1.7 90) (layer F.Fab) hide
+    (fp_text value 100k (at 0.6 1.7 90) (layer F.Fab) hide
       (effects (font (size 1 1) (thickness 0.15)))
     )
@@
       (effects (font (size 0.5 0.5) (thickness 0.125)))
     )
-    (fp_text value resistor (at 0.6 1.7 90) (layer F.Fab) hide
+    (fp_text value 100 (at 0.6 1.7 90) (layer F.Fab) hide
       (effects (font (size 1 1) (thickness 0.15)))
     )
@@
       (effects (font (size 0.5 0.5) (thickness 0.125)))
     )
-    (fp_text value resistor (at 0.6 1.7) (layer F.Fab) hide
+    (fp_text value 100 (at 0.6 1.7) (layer F.Fab) hide
       (effects (font (size 1 1) (thickness 0.15)))
     )
@@
       (effects (font (size 0.5 0.5) (thickness 0.125)))
     )
-    (fp_text value resistor (at 0.6 1.7 180) (layer F.Fab) hide
+    (fp_text value 100 (at 0.6 1.7 180) (layer F.Fab) hide
       (effects (font (size 1 1) (thickness 0.15)))
     )
@@
       (effects (font (size 0.5 0.5) (thickness 0.125)))
     )
-    (fp_text value capacitor (at 0.6 1.7 90) (layer F.Fab) hide
+    (fp_text value 0.1 (at 0.6 1.7 90) (layer F.Fab) hide
       (effects (font (size 1 1) (thickness 0.15)))
     )
@@
       (effects (font (size 0.5 0.5) (thickness 0.125)))
     )
-    (fp_text value capacitor (at 0.6 1.7) (layer F.Fab) hide
+    (fp_text value 0.1 (at 0.6 1.7) (layer F.Fab) hide
       (effects (font (size 1 1) (thickness 0.15)))
     )
@@
       (effects (font (size 0.5 0.5) (thickness 0.125)))
     )
-    (fp_text value resistor (at 0.6 1.7) (layer F.Fab) hide
+    (fp_text value 1k (at 0.6 1.7) (layer F.Fab) hide
       (effects (font (size 1 1) (thickness 0.15)))
     )
@@
       (effects (font (size 0.5 0.5) (thickness 0.125)))
     )
-    (fp_text value resistor (at 0.6 1.7 270) (layer F.Fab) hide
+    (fp_text value 1k (at 0.6 1.7 270) (layer F.Fab) hide
       (effects (font (size 1 1) (thickness 0.15)))
     )
@@
       (effects (font (size 0.5 0.5) (thickness 0.125)))
     )
-    (fp_text value 390k (at 0.6 1.7 180) (layer F.Fab) hide
+    (fp_text value 10k (at 0.6 1.7 180) (layer F.Fab) hide
       (effects (font (size 1 1) (thickness 0.15)))
     )
@@
       (effects (font (size 0.5 0.5) (thickness 0.125)))
     )
-    (fp_text value 390k (at 0.6 1.7 180) (layer F.Fab) hide
-      (effects (font (size 1 1) (thickness 0.15)))
-    )
+    (fp_text value 10k (at 0.6 1.7 180) (layer F.Fab) hide
+      (effects (font (size 1 1) (thickness 0.15)))
+    )

Commit message: PCB component values update
Parts:
- C10, C12, C13, C14, C20, C5, C9: value capacitor -> 0.1
- C11: value capacitor -> 22u
- R10: value resistor -> 1k
- R5, R8, R9: value resistor -> 10k
Changed lines of the file:
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@@
-(kicad_pcb (version 4) (host pcbnew "(2016-04-26 BZR 6712, Git b92ad6f)-product")
+(kicad_pcb (version 4) (host pcbnew "(2016-06-02 BZR 6871, Git 368bd14)-product")
   (general
     (links 193)
@@
       (effects (font (size 0.5 0.5) (thickness 0.125)))
     )
-    (fp_text value resistor (at 0.6 1.7 270) (layer F.Fab) hide
+    (fp_text value 10k (at 0.6 1.7 270) (layer F.Fab) hide
       (effects (font (size 1 1) (thickness 0.15)))
     )
@@
       (effects (font (size 0.5 0.5) (thickness 0.125)))
     )
-    (fp_text value capacitor (at 0.6 1.7) (layer F.Fab) hide
+    (fp_text value 0.1 (at 0.6 1.7) (layer F.Fab) hide
       (effects (font (size 1 1) (thickness 0.15)))
     )
@@
       (effects (font (size 0.5 0.5) (thickness 0.125)))
     )
-    (fp_text value resistor (at 0.6 1.7 270) (layer F.Fab) hide
+    (fp_text value 10k (at 0.6 1.7 270) (layer F.Fab) hide
       (effects (font (size 1 1) (thickness 0.15)))
     )
@@
       (effects (font (size 0.5 0.5) (thickness 0.125)))
     )
-    (fp_text value resistor (at 0.6 1.7) (layer F.Fab) hide
+    (fp_text value 10k (at 0.6 1.7) (layer F.Fab) hide
       (effects (font (size 1 1) (thickness 0.15)))
     )
@@
       (effects (font (size 0.5 0.5) (thickness 0.125)))
     )
-    (fp_text value capacitor (at 0.6 1.7 90) (layer F.Fab) hide
+    (fp_text value 0.1 (at 0.6 1.7 90) (layer F.Fab) hide
       (effects (font (size 1 1) (thickness 0.15)))
     )
@@
       (effects (font (size 0.5 0.5) (thickness 0.125)))
     )
-    (fp_text value capacitor (at 0.6 1.7 90) (layer F.Fab) hide
+    (fp_text value 0.1 (at 0.6 1.7 90) (layer F.Fab) hide
       (effects (font (size 1 1) (thickness 0.15)))
     )
@@
       (effects (font (size 0.5 0.5) (thickness 0.125)))
     )
-    (fp_text value capacitor (at 0.6 1.7 180) (layer F.Fab) hide
+    (fp_text value 0.1 (at 0.6 1.7 180) (layer F.Fab) hide
       (effects (font (size 1 1) (thickness 0.15)))
     )
@@
       (effects (font (size 0.5 0.5) (thickness 0.125)))
     )
-    (fp_text value capacitor (at 0.6 1.7 90) (layer F.Fab) hide
+    (fp_text value 0.1 (at 0.6 1.7 90) (layer F.Fab) hide
       (effects (font (size 1 1) (thickness 0.15)))
     )
@@
       (effects (font (size 0.5 0.5) (thickness 0.125)))
     )
-    (fp_text value capacitor (at 0.6 1.7) (layer F.Fab) hide
+    (fp_text value 0.1 (at 0.6 1.7) (layer F.Fab) hide
       (effects (font (size 1 1) (thickness 0.15)))
     )
@@
       (effects (font (size 0.5 0.5) (thickness 0.125)))
     )
-    (fp_text value resistor (at 0.6 1.7 90) (layer F.Fab) hide
+    (fp_text value 1k (at 0.6 1.7 90) (layer F.Fab) hide
       (effects (font (size 1 1) (thickness 0.15)))
     )
@@
       (effects (font (size 0.5 0.5) (thickness 0.125)))
     )
-    (fp_text value capacitor (at 0.6 1.7 180) (layer F.Fab) hide
+    (fp_text value 22u (at 0.6 1.7 180) (layer F.Fab) hide
       (effects (font (size 1 1) (thickness 0.15)))
     )
@@
       (effects (font (size 0.5 0.5) (thickness 0.125)))
     )
-    (fp_text value capacitor (at 0.6 1.7) (layer F.Fab) hide
-      (effects (font (size 1 1) (thickness 0.15)))
-    )
+    (fp_text value 0.1 (at 0.6 1.7) (layer F.Fab) hide
+      (effects (font (size 1 1) (thickness 0.15)))
+    )

Commit message: Closes #10 (migration to 128kB flash)
Parts:
- U1: value STM32F103C8T6 -> STM32F103CBT6
- XC1: value CRYSTAL_4pin -> 16MHz
Changed lines of the file:
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@@
-(kicad_pcb (version 4) (host pcbnew "(2016-06-02 BZR 6871, Git 368bd14)-product")
+(kicad_pcb (version 4) (host pcbnew "(2016-06-30 BZR 6960, Git 6614e5e)-product")
   (general
     (links 193)
@@
       (effects (font (size 0.8 0.8) (thickness 0.16)))
     )
-    (fp_text value STM32F103C8T6 (at 3.75 -5) (layer F.Fab) hide
+    (fp_text value STM32F103CBT6 (at 3.75 -5) (layer F.Fab) hide
       (effects (font (size 1 1) (thickness 0.15)))
     )
@@
       (effects (font (size 1 1) (thickness 0.15)))
     )
-    (fp_text value CRYSTAL_4pin (at 0.9 -3.3) (layer F.Fab) hide
+    (fp_text value 16MHz (at 0.9 -3.3) (layer F.Fab) hide
       (effects (font (size 1 1) (thickness 0.15)))
     )
